File: hardware/active_power/ltc3108_power_breakout.kicad_pcb (KiCad board)
At the start: 2 copper layers, 77 x 57 mm, 13 parts, among them J1 TEG, J2 External_LPR6235_752SML, J3 OUT_3V3_LAB, J4 EXTERNAL_VSTORE_SUPERCAP_6V3, J5 PGOOD_MONITOR, U1 LTC3108EGN

Commit message: legal: reserve Mojeaterego Andrzej Mikulski rights and publish authorized contact across project artifacts
Other:
- board text added: "MOJEATEREGO (C) 2026 A. MIKULSKI"
Changed lines of the file:
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@@
 (gr_line (start 87 67) (end 10 67) (stroke (width 0.05) (type default)) (layer "Edge.Cuts"))
 (gr_line (start 10 67) (end 10 10) (stroke (width 0.05) (type default)) (layer "Edge.Cuts"))
+(gr_text "MOJEATEREGO (C) 2026 A. MIKULSKI" (at 48 58) (layer "B.SilkS") (effects (font (size 0.85 0.85) (thickness 0.13))))
 (gr_text "LTC3108 LAB POWER / UNROUTED REV A0" (at 46 63) (layer "F.SilkS") (effects (font (size 1 1) (thickness 0.15))))
 )
