File: hardware/kicad/thermo_bench_carrier.kicad_pcb (KiCad board)
At the start: 2 copper layers, 70 x 44 mm, 5 parts, among them J1 EXT_BENCH_3V3, J2 WIO_E5_DEV_UART, J3 USB_UART_3V3, J4 RAW_TEG_PROBE, J5 PMIC_OUTPUT_PROBE

Commit message: legal: reserve Mojeaterego Andrzej Mikulski rights and publish authorized contact across project artifacts
Other:
- board text added: "MOJEATEREGO (C) 2026 A. MIKULSKI"
Changed lines of the file:
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@@
 (gr_line (start 82 57) (end 12 57) (stroke (width 0.05) (type default)) (layer "Edge.Cuts"))
 (gr_line (start 12 57) (end 12 13) (stroke (width 0.05) (type default)) (layer "Edge.Cuts"))
+(gr_text "MOJEATEREGO (C) 2026 A. MIKULSKI" (at 47 49.2) (layer "B.SilkS") (effects (font (size 0.85 0.85) (thickness 0.13))))
  (gr_text "THERMO-IOT LAB CARRIER REV A0" (at 47 53) (layer "F.SilkS") (effects (font (size 1.15 1.15) (thickness 0.15))))
  (gr_text "PMIC + TEG PROBES ISOLATED" (at 60 46) (layer "F.SilkS") (effects (font (size 1 1) (thickness 0.15))))
